Commit message: adding urdf

File: arha_description/urdf/ARHA.urdf (robot description, URDF)
Before this commit: robot arha_description, 15 links, 14 joints
Links:
- link base_link: mass 0.646806335459542 -> 50.0
Joints:
- joint WristLU_joint: limit lower=-1.5708 upper=1.5708 effort=20 velocity=0 -> lower=-1.5708 upper=1.5708 effort=20 velocity=19.897
- joint WristRU_joint: limit lower=-1.5708 upper=1.5708 effort=20 velocity=0 -> lower=-1.5708 upper=1.5708 effort=20 velocity=19.897

Commit message: adding current code for gravity compensation and masses updated from the robot's urdf

File: arha_description/urdf/ARHA.urdf (robot description, URDF)
Before this commit: robot arha_description, 15 links, 14 joints
Links:
- added link ElbowLD_motor5_link, mass 0.0
- added link ElbowLU_motor3_link, mass 0.0
- added link ElbowLU_motor4_link, mass 0.0
- added link ElbowRD_motor5_link, mass 0.0
- added link ElbowRU_motor3_link, mass 0.0
- added link ElbowRU_motor4_link, mass 0.0
- added link ShoulderLU_motor2_link, mass 0.0
- added link ShoulderRU_motor2_link, mass 0.0
- added link WristLD_motor6_link, mass 0.0
- added link WristRD_motor6_link, mass 0.0
- link ElbowLD_link: mass 0.405367875717028 -> 1.05401
- link ElbowLU_link: mass 0.435431174027291 -> 1.9519
- link ElbowRD_link: mass 0.405367838897484 -> 1.05401
- link ElbowRU_link: mass 0.43543149660162 -> 1.9519
- link ShoulderLD_link: mass 0.121271829639387 -> 0.12
- link ShoulderLU_link: mass 0.437859352194871 -> 1.36249
- link ShoulderRD_link: mass 0.121271833885802 -> 0.12
- link ShoulderRU_link: mass 0.437859351944568 -> 1.36249
- link WristLD_link: mass 0.144157848422193 -> 0.7646
- link WristLU_link: mass 0.348222374397224 -> 0.1
- link WristRD_link: mass 0.144157843696757 -> 0.7646
- link WristRU_link: mass 0.348222354843636 -> 0.1
Joints:
- added joint ElbowLD_motor5_fixed: type fixed, parent ElbowLD_link, child ElbowLD_motor5_link, origin xyz=0.033161 -0.0056591 -0.11391 rpy=0 0 0
- added joint ElbowLU_motor3_fixed: type fixed, parent ElbowLU_link, child ElbowLU_motor3_link, origin xyz=0 0 0 rpy=0 0 0
- added joint ElbowLU_motor4_fixed: type fixed, parent ElbowLU_link, child ElbowLU_motor4_link, origin xyz=0.075262 -0.00045791 -0.2413 rpy=0 0 0
- added joint ElbowRD_motor5_fixed: type fixed, parent ElbowRD_link, child ElbowRD_motor5_link, origin xyz=0.032837 -0.0055583 -0.1128 rpy=0 0 0
- added joint ElbowRU_motor3_fixed: type fixed, parent ElbowRU_link, child ElbowRU_motor3_link, origin xyz=0 0 0 rpy=0 0 0
- added joint ElbowRU_motor4_fixed: type fixed, parent ElbowRU_link, child ElbowRU_motor4_link, origin xyz=0.079705 -0.00060472 -0.23692 rpy=0 0 0
- added joint ShoulderLU_motor2_fixed: type fixed, parent ShoulderLU_link, child ShoulderLU_motor2_link, origin xyz=0 0.086954 0 rpy=0 0 0
- added joint ShoulderRU_motor2_fixed: type fixed, parent ShoulderRU_link, child ShoulderRU_motor2_link, origin xyz=0 0.091943 0 rpy=0 0 0
- added joint WristLD_motor6_fixed: type fixed, parent WristLD_link, child WristLD_motor6_link, origin xyz=0 0 0 rpy=0 0 0
- added joint WristRD_motor6_fixed: type fixed, parent WristRD_link, child WristRD_motor6_link, origin xyz=0 0 0 rpy=0 0 0

File: arha_moveit2/config/arha_description.ros2_control.xacro (robot description, xacro)
@@ -13,4 +13,10 @@
                     <param name="port">5000</param>
                     <param name="zero_on_startup">${zero_on_startup}</param>
+                    <param name="gravity_compensation">true</param>
+                    <param name="left_arm_base_link">chest_link</param>
+                    <param name="left_arm_tip_link">WristLD_link</param>
+                    <param name="right_arm_base_link">chest_link</param>
+                    <param name="right_arm_tip_link">WristRD_link</param>
+                    <param name="urdf_path">$(find arha_description)/urdf/ARHA.urdf</param>
                 </xacro:unless>
             </hardware>
