Commit message: updating progress

File: arha_description/urdf/ARHA.urdf (robot description, URDF)
Before this commit: robot arha_description, 25 links, 24 joints
Links:
- link ElbowLD_link: geometry visual mesh filename=package://arha_description/meshes/ElbowLD_link.STL
- link ElbowLU_link: geometry visual mesh filename=package://arha_description/meshes/ElbowLU_link.STL
- link ElbowRD_link: geometry visual mesh filename=package://arha_description/meshes/ElbowRD_link.STL
- link ElbowRD_motor5_link: mass 0.0 -> 0.01
- link ElbowRU_link: geometry visual mesh filename=package://arha_description/meshes/ElbowRU_link.STL
- link ShoulderLD_link: geometry visual mesh filename=package://arha_description/meshes/ShoulderLD_link.STL
- link ShoulderLU_link: geometry visual mesh filename=package://arha_description/meshes/ShoulderLU_link.STL
- link ShoulderRD_link: geometry visual mesh filename=package://arha_description/meshes/ShoulderRD_link.STL
- link ShoulderRU_link: geometry visual mesh filename=package://arha_description/meshes/ShoulderRU_link.STL
- link WristLD_link: geometry visual mesh filename=package://arha_description/meshes/WristLD_link.STL
- link WristLU_link: geometry visual mesh filename=package://arha_description/meshes/WristLU_link.STL
- link WristRD_link: mass 0.7646 -> 1.36; geometry visual mesh filename=package://arha_description/meshes/WristRD_link.STL
- link WristRD_motor6_link: mass 0.0 -> 0.01
- link WristRU_link: geometry visual mesh filename=package://arha_description/meshes/WristRU_link.STL
Joints:
- joint ElbowLD_joint: limit lower=-1.5708 upper=0 effort=60 velocity=4.1888 -> lower=-1.5708 upper=0 effort=5000 velocity=4.1888
- joint ElbowLU_joint: limit lower=-1.5708 upper=1.5708 effort=20 velocity=19.897 -> lower=-1.5708 upper=1.5708 effort=5000 velocity=19.897
- joint ElbowRD_joint: limit lower=0 upper=1.5708 effort=60 velocity=4.1888 -> lower=0 upper=1.5708 effort=5000 velocity=4.1888
- joint ElbowRU_joint: limit lower=-1.5708 upper=1.5708 effort=20 velocity=19.897 -> lower=-1.5708 upper=1.5708 effort=5000 velocity=19.897
- joint ShoulderLD_joint: limit lower=0 upper=1.5708 effort=60 velocity=4.1888 -> lower=0 upper=1.5708 effort=5000 velocity=4.1888
- joint ShoulderLU_joint: limit lower=-1.5708 upper=1.5708 effort=100 velocity=5.235988 -> lower=-1.5708 upper=1.5708 effort=5000 velocity=5.235988
- joint ShoulderRD_joint: limit lower=-1.5708 upper=0 effort=60 velocity=4.1888 -> lower=-1.5708 upper=0 effort=5000 velocity=4.1888
- joint ShoulderRU_joint: limit lower=-1.5708 upper=1.5708 effort=100 velocity=5.235988 -> lower=-1.5708 upper=1.5708 effort=5000 velocity=5.235988
- joint WristLD_joint: limit lower=-1.5708 upper=1.5708 effort=8 velocity=32.463124 -> lower=-1.5708 upper=1.5708 effort=5000 velocity=32.463124
- joint WristLU_joint: limit lower=-1.5708 upper=1.5708 effort=20 velocity=19.897 -> lower=-1.5708 upper=1.5708 effort=5000 velocity=19.897
- joint WristRD_joint: limit lower=-1.5708 upper=1.5708 effort=8 velocity=32.463 -> lower=-1.5708 upper=1.5708 effort=5000 velocity=32.463
- joint WristRU_joint: limit lower=-1.5708 upper=1.5708 effort=20 velocity=19.897 -> lower=-1.5708 upper=1.5708 effort=5000 velocity=19.897

File: arha_gazebo/urdf/arha_with_grippers.urdf.xacro (robot description, xacro)
@@ -41,6 +41,6 @@
       <geometry>
         <cylinder>
-          <radius>0.05</radius>
-          <length>0.15</length>
+          <radius>0.04</radius>
+          <length>0.12</length>
         </cylinder>
       </geometry>
@@ -51,6 +51,6 @@
       <geometry>
         <cylinder>
-          <radius>0.05</radius>
-          <length>0.20</length>
+          <radius>0.04</radius>
+          <length>0.16</length>
         </cylinder>
       </geometry>
@@ -61,6 +61,6 @@
       <geometry>
         <cylinder>
-          <radius>0.04</radius>
-          <length>0.12</length>
+          <radius>0.03</radius>
+          <length>0.10</length>
         </cylinder>
       </geometry>
@@ -71,6 +71,6 @@
       <geometry>
         <cylinder>
-          <radius>0.04</radius>
-          <length>0.25</length>
+          <radius>0.03</radius>
+          <length>0.20</length>
         </cylinder>
       </geometry>
@@ -81,6 +81,6 @@
       <geometry>
         <cylinder>
-          <radius>0.03</radius>
-          <length>0.08</length>
+          <radius>0.02</radius>
+          <length>0.06</length>
         </cylinder>
       </geometry>
@@ -91,6 +91,6 @@
       <geometry>
         <cylinder>
-          <radius>0.03</radius>
-          <length>0.10</length>
+          <radius>0.02</radius>
+          <length>0.08</length>
         </cylinder>
       </geometry>
@@ -102,6 +102,6 @@
       <geometry>
         <cylinder>
-          <radius>0.05</radius>
-          <length>0.15</length>
+          <radius>0.04</radius>
+          <length>0.12</length>
         </cylinder>
       </geometry>
@@ -112,6 +112,6 @@
       <geometry>
         <cylinder>
-          <radius>0.05</radius>
-          <length>0.20</length>
+          <radius>0.04</radius>
+          <length>0.16</length>
         </cylinder>
       </geometry>
@@ -122,6 +122,6 @@
       <geometry>
         <cylinder>
-          <radius>0.04</radius>
-          <length>0.12</length>
+          <radius>0.03</radius>
+          <length>0.10</length>
         </cylinder>
       </geometry>
@@ -132,6 +132,6 @@
       <geometry>
         <cylinder>
-          <radius>0.04</radius>
-          <length>0.25</length>
+          <radius>0.03</radius>
+          <length>0.20</length>
         </cylinder>
       </geometry>
@@ -142,6 +142,6 @@
       <geometry>
         <cylinder>
-          <radius>0.03</radius>
-          <length>0.08</length>
+          <radius>0.02</radius>
+          <length>0.06</length>
         </cylinder>
       </geometry>
@@ -152,6 +152,6 @@
       <geometry>
         <cylinder>
-          <radius>0.03</radius>
-          <length>0.10</length>
+          <radius>0.02</radius>
+          <length>0.08</length>
         </cylinder>
       </geometry>
@@ -169,4 +169,8 @@
         <param name="max">3.14</param>
       </command_interface>
+      <command_interface name="effort">
+        <param name="min">-1000</param>
+        <param name="max">1000</param>
+      </command_interface>
       <state_interface name="position"/>
       <state_interface name="velocity"/>
@@ -177,4 +181,8 @@
         <param name="max">3.14</param>
       </command_interface>
+      <command_interface name="effort">
+        <param name="min">-1000</param>
+        <param name="max">1000</param>
+      </command_interface>
       <state_interface name="position"/>
       <state_interface name="velocity"/>
@@ -185,4 +193,8 @@
         <param name="max">3.14</param>
       </command_interface>
+      <command_interface name="effort">
+        <param name="min">-1000</param>
+        <param name="max">1000</param>
+      </command_interface>
       <state_interface name="position"/>
       <state_interface name="velocity"/>
@@ -193,4 +205,8 @@
         <param name="max">3.14</param>
       </command_interface>
+      <command_interface name="effort">
+        <param name="min">-1000</param>
+        <param name="max">1000</param>
+      </command_interface>
       <state_interface name="position"/>
       <state_interface name="velocity"/>
@@ -201,4 +217,8 @@
         <param name="max">3.14</param>
       </command_interface>
+      <command_interface name="effort">
+        <param name="min">-1000</param>
+        <param name="max">1000</param>
+      </command_interface>
       <state_interface name="position"/>
       <state_interface name="velocity"/>
@@ -208,4 +228,8 @@
         <param name="min">-3.14</param>
         <param name="max">3.14</param>
+      </command_interface>
+      <command_interface name="effort">
+        <param name="min">-1000</param>
+        <param name="max">1000</param>
       </command_interface>
       <state_interface name="position"/>
@@ -218,4 +242,8 @@
         <param name="max">3.14</param>
       </command_interface>
+      <command_interface name="effort">
+        <param name="min">-1000</param>
+        <param name="max">1000</param>
+      </command_interface>
       <state_interface name="position"/>
       <state_interface name="velocity"/>
@@ -226,4 +254,8 @@
         <param name="max">3.14</param>
       </command_interface>
+      <command_interface name="effort">
+        <param name="min">-1000</param>
+        <param name="max">1000</param>
+      </command_interface>
       <state_interface name="position"/>
       <state_interface name="velocity"/>
@@ -234,4 +266,8 @@
         <param name="max">3.14</param>
       </command_interface>
+      <command_interface name="effort">
+        <param name="min">-1000</param>
+        <param name="max">1000</param>
+      </command_interface>
       <state_interface name="position"/>
       <state_interface name="velocity"/>
@@ -242,4 +278,8 @@
         <param name="max">3.14</param>
       </command_interface>
+      <command_interface name="effort">
+        <param name="min">-1000</param>
+        <param name="max">1000</param>
+      </command_interface>
       <state_interface name="position"/>
       <state_interface name="velocity"/>
@@ -250,4 +290,8 @@
         <param name="max">3.14</param>
       </command_interface>
+      <command_interface name="effort">
+        <param name="min">-1000</param>
+        <param name="max">1000</param>
+      </command_interface>
       <state_interface name="position"/>
       <state_interface name="velocity"/>
@@ -258,20 +302,16 @@
         <param name="max">3.14</param>
       </command_interface>
+      <command_interface name="effort">
+        <param name="min">-1000</param>
+        <param name="max">1000</param>
+      </command_interface>
       <state_interface name="position"/>
       <state_interface name="velocity"/>
     </joint>
     <!-- Left Gripper Joints -->
-    <joint name="left_robotiq_hande_left_finger_joint">
-      <command_interface name="position">
-        <param name="min">0.0</param>
-        <param name="max">0.025</param>
-      </command_interface>
-      <state_interface name="position"/>
-      <state_interface name="velocity"/>
-    </joint>
-    <joint name="left_robotiq_hande_right_finger_joint">
-      <command_interface name="position">
-        <param name="min">0.0</param>
-        <param name="max">0.025</param>
+    <joint name="left_cam_joint">
+      <command_interface name="position">
+        <param name="min">-0.57</param>
+        <param name="max">0.0</param>
       </command_interface>
       <state_interface name="position"/>
@@ -279,16 +319,8 @@
     </joint>
     <!-- Right Gripper Joints -->
-    <joint name="right_robotiq_hande_left_finger_joint">
-      <command_interface name="position">
-        <param name="min">0.0</param>
-        <param name="max">0.025</param>
-      </command_interface>
-      <state_interface name="position"/>
-      <state_interface name="velocity"/>
-    </joint>
-    <joint name="right_robotiq_hande_right_finger_joint">
-      <command_interface name="position">
-        <param name="min">0.0</param>
-        <param name="max">0.025</param>
+    <joint name="right_cam_joint">
+      <command_interface name="position">
+        <param name="min">-0.57</param>
+        <param name="max">0.0</param>
       </command_interface>
       <state_interface name="position"/>

File: arha_gazebo/urdf/grippers/left_gripper_mount.xacro (robot description, xacro)
@@ -1,45 +1,15 @@
 <?xml version="1.0"?>
 <robot xmlns:xacro="http://www.ros.org/wiki/xacro">
-  <!-- Include the Robotiq Hand-E gripper -->
-  <xacro:include filename="$(find robotiq_hande_description)/urdf/robotiq_hande_gripper.xacro"/>
-  <!-- Instantiate left gripper (ros2_control disabled for Gazebo Classic) -->
-  <xacro:robotiq_hande_gripper
-    name="left_gripper"
-    prefix="left_"
+  <!-- Left Gripper Mount -->
+  <xacro:include filename="$(find arha_gazebo)/urdf/grippers/pincopen.xacro"/>
+  <xacro:include filename="$(find realsense2_description)/urdf/_d435.urdf.xacro" />
+  <xacro:pincopen_gripper
+    prefix="left"
     parent="WristLD_link"
-    grip_pos_min="0.0"
-    grip_pos_max="0.025"
-    tty_port="/dev/null"
-    baudrate="115200"
-    parity="N"
-    data_bits="8"
-    stop_bit="1"
-    slave_id="9"
-    use_fake_hardware="true"
-    xyz="0 0 0.06"
-    rpy="0 0 0"
-    use_mimic="false"
-    use_ros2_control="false"
-  />
-  <!-- NOTE: ros2_control for gripper joints is defined in arha_with_grippers.urdf.xacro
-       to avoid duplicate ros2_control blocks in Gazebo Classic -->
-  <!-- Add gazebo_grasp_fix plugin for grasping objects -->
-  <!--
-  <gazebo>
-     <plugin name="left_gripper_grasp" filename="libgazebo_grasp_fix.so">
-      <arm>
-        <arm_name>left_gripper</arm_name>
-        <palm_link>left_robotiq_hande_link</palm_link>
-        <gripper_link>left_robotiq_hande_left_finger</gripper_link>
-        <gripper_link>left_robotiq_hande_right_finger</gripper_link>
-      </arm>
-      <forces_angle_tolerance>100</forces_angle_tolerance>
-      <update_rate>4</update_rate>
-      <grip_count_threshold>4</grip_count_threshold>
-      <max_grip_count>8</max_grip_count>
-      <release_tolerance>0.005</release_tolerance>
-      <disable_collisions_on_attach>false</disable_collisions_on_attach>
-    </plugin>
-  </gazebo>
-  -->
+  >
+    <origin xyz="0 0 0.13" rpy="1.5708 -1.5708 3.14159" />
+  </xacro:pincopen_gripper>
+  <xacro:sensor_d435 parent="left_Camera_mount_V1" name="left_camera" use_nominal_extrinsics="false" add_plug="false" use_mesh="true">
+    <origin xyz="0 0 0" rpy="0 0 1.5708"/>
+  </xacro:sensor_d435>
 </robot>

File: arha_gazebo/urdf/grippers/right_gripper_mount.xacro (robot description, xacro)
@@ -1,45 +1,15 @@
 <?xml version="1.0"?>
 <robot xmlns:xacro="http://www.ros.org/wiki/xacro">
-  <!-- Include the Robotiq Hand-E gripper -->
-  <xacro:include filename="$(find robotiq_hande_description)/urdf/robotiq_hande_gripper.xacro"/>
-  <!-- Instantiate right gripper (ros2_control disabled for Gazebo Classic) -->
-  <xacro:robotiq_hande_gripper
-    name="right_gripper"
-    prefix="right_"
+  <!-- Right Gripper Mount -->
+  <xacro:include filename="$(find arha_gazebo)/urdf/grippers/pincopen.xacro"/>
+  <xacro:include filename="$(find realsense2_description)/urdf/_d435.urdf.xacro" />
+  <xacro:pincopen_gripper
+    prefix="right"
     parent="WristRD_link"
-    grip_pos_min="0.0"
-    grip_pos_max="0.025"
-    tty_port="/dev/null"
-    baudrate="115200"
-    parity="N"
-    data_bits="8"
-    stop_bit="1"
-    slave_id="10"
-    use_fake_hardware="true"
-    xyz="0 0 0.06"
-    rpy="0 0 0"
-    use_mimic="false"
-    use_ros2_control="false"
-  />
-  <!-- NOTE: ros2_control for gripper joints is defined in arha_with_grippers.urdf.xacro
-       to avoid duplicate ros2_control blocks in Gazebo Classic -->
-  <!-- Add gazebo_grasp_fix plugin for grasping objects (commented out for now) -->
-  <!--
-  <gazebo>
-    <plugin name="right_gripper_grasp" filename="libgazebo_grasp_fix.so">
-      <arm>
-        <arm_name>right_gripper</arm_name>
-        <palm_link>right_robotiq_hande_link</palm_link>
-        <gripper_link>right_robotiq_hande_left_finger</gripper_link>
-        <gripper_link>right_robotiq_hande_right_finger</gripper_link>
-      </arm>
-      <forces_angle_tolerance>100</forces_angle_tolerance>
-      <update_rate>4</update_rate>
-      <grip_count_threshold>4</grip_count_threshold>
-      <max_grip_count>8</max_grip_count>
-      <release_tolerance>0.005</release_tolerance>
-      <disable_collisions_on_attach>false</disable_collisions_on_attach>
-    </plugin>
-  </gazebo>
-  -->
+  >
+    <origin xyz="0 0 0.13" rpy="1.5708 -1.5708 0.0" />
+  </xacro:pincopen_gripper>
+  <xacro:sensor_d435 parent="right_Camera_mount_V1" name="right_camera" use_nominal_extrinsics="false" add_plug="false" use_mesh="true">
+    <origin xyz="0 0 0" rpy="0 0 1.5708"/>
+  </xacro:sensor_d435>
 </robot>

File: arha_moveit2/config/arha_description.ros2_control.xacro (robot description, xacro)
@@ -21,5 +21,5 @@
                 </xacro:unless>
             </hardware>
-            <!-- LEFT ARM JOINTS -->
+            <!-- Left Arm -->
             <joint name="ShoulderLU_joint">
                 <command_interface name="position"/>
@@ -88,5 +88,5 @@
                 <param name="direction">-1</param>
             </joint>
-            <!-- RIGHT ARM JOINTS -->
+            <!-- Right Arm -->
             <joint name="ShoulderRU_joint">
                 <command_interface name="position"/>
@@ -155,4 +155,27 @@
                 <param name="direction">-1</param>
             </joint>
+            <!-- Gripper -->
+            <joint name="left_cam_joint">
+                <command_interface name="position"/>
+                <state_interface name="position">
+                  <param name="initial_value">0.0</param>
+                </state_interface>
+                <state_interface name="velocity"/>
+                <state_interface name="effort"/>
+                <param name="limb_name">left_gripper</param>
+                <param name="motor_id">2</param>
+                <param name="direction">1</param>
+            </joint>
+            <joint name="right_cam_joint">
+                <command_interface name="position"/>
+                <state_interface name="position">
+                  <param name="initial_value">0.0</param>
+                </state_interface>
+                <state_interface name="velocity"/>
+                <state_interface name="effort"/>
+                <param name="limb_name">right_gripper</param>
+                <param name="motor_id">1</param>
+                <param name="direction">1</param>
+            </joint>
         </ros2_control>
     </xacro:macro>

File: arha_moveit2/config/arha_description.ros2_control_right_arm.xacro (robot description, xacro)
@@ -15,5 +15,5 @@
                 </xacro:unless>
             </hardware>
-            <!-- RIGHT ARM JOINTS -->
+            <!-- Right Arm -->
             <joint name="ShoulderRU_joint">
                 <command_interface name="position"/>
@@ -82,4 +82,16 @@
                 <param name="direction">1</param>
             </joint>
+            <!-- Gripper -->
+            <joint name="right_cam_joint">
+                <command_interface name="position"/>
+                <state_interface name="position">
+                  <param name="initial_value">0.0</param>
+                </state_interface>
+                <state_interface name="velocity"/>
+                <state_interface name="effort"/>
+                <param name="limb_name">right_gripper</param>
+                <param name="motor_id">1</param>
+                <param name="direction">1</param>
+            </joint>
         </ros2_control>
     </xacro:macro>

File: arha_moveit2/config/arha_description.urdf.xacro (robot description, xacro)
@@ -4,7 +4,22 @@
     <xacro:arg name="use_fake_hardware" default="true" />
     <xacro:arg name="zero_on_startup" default="false" />
-    <!-- Import arha_description urdf file -->
+    <!-- URDF Include -->
     <xacro:include filename="$(find arha_description)/urdf/ARHA.urdf" />
-    <!-- Import control_xacro -->
+    <!-- Gripper and Camera Assembly -->
+    <xacro:include filename="$(find arha_gazebo)/urdf/grippers/pincopen.xacro"/>
+    <xacro:include filename="$(find realsense2_description)/urdf/_d435.urdf.xacro" />
+    <xacro:pincopen_gripper prefix="left" parent="WristLD_link">
+      <origin xyz="0 0 0.13" rpy="1.5708 -1.5708 3.14159" />
+    </xacro:pincopen_gripper>
+    <xacro:sensor_d435 parent="left_Camera_mount_V1" name="left_camera" use_nominal_extrinsics="false" add_plug="false" use_mesh="true">
+      <origin xyz="-0.01 -0.008 0.011" rpy="0 0 1.5708"/>
+    </xacro:sensor_d435>
+    <xacro:pincopen_gripper prefix="right" parent="WristRD_link">
+      <origin xyz="0 0 0.13" rpy="1.5708 -1.5708 0.0" />
+    </xacro:pincopen_gripper>
+    <xacro:sensor_d435 parent="right_Camera_mount_V1" name="right_camera" use_nominal_extrinsics="false" add_plug="false" use_mesh="true">
+      <origin xyz="-0.01 -0.008 0.011" rpy="0 0 1.5708"/>
+    </xacro:sensor_d435>
+    <!-- Control Include -->
     <xacro:include filename="arha_description.ros2_control.xacro" />
     <xacro:arha_description_ros2_control name="ARHA" initial_positions_file="$(arg initial_positions_file)" use_fake_hardware="$(arg use_fake_hardware)" zero_on_startup="$(arg zero_on_startup)"/>

File: arha_moveit2/config/arha_description_right_arm.urdf.xacro (robot description, xacro)
@@ -3,7 +3,16 @@
     <xacro:arg name="initial_positions_file" default="initial_positions.yaml" />
     <xacro:arg name="use_fake_hardware" default="true" />
-    <!-- Import arha_description urdf file (dual arm) -->
+    <!-- URDF Include -->
     <xacro:include filename="$(find arha_description)/urdf/ARHA.urdf" />
-    <!-- Import right arm control_xacro -->
+    <!-- Gripper and Camera Assembly -->
+    <xacro:include filename="$(find arha_gazebo)/urdf/grippers/pincopen.xacro"/>
+    <xacro:include filename="$(find realsense2_description)/urdf/_d435.urdf.xacro" />
+    <xacro:pincopen_gripper prefix="right" parent="WristRD_link">
+      <origin xyz="0 0 0.13" rpy="1.5708 -1.5708 0.0" />
+    </xacro:pincopen_gripper>
+    <xacro:sensor_d435 parent="right_Camera_mount_V1" name="right_camera" use_nominal_extrinsics="false" add_plug="false" use_mesh="true">
+      <origin xyz="0 0 0" rpy="0 0 1.5708"/>
+    </xacro:sensor_d435>
+    <!-- Control Include -->
     <xacro:include filename="arha_description.ros2_control_right_arm.xacro" />
     <!-- Configure ros2_control for right arm only -->
