Commit message: refactor: changes related to gazebo and moveit2 for virtual simulation of new grippers and controllers.

File: arha_description/urdf/ARHA.urdf (robot description, URDF)
Before this commit: robot arha_description, 25 links, 24 joints
Links:
- link ElbowLD_link: geometry collision mesh filename=package://arha_description/meshes/ElbowLD_link.STL; visual mesh filename=package://arha_description/meshes/ElbowLD_link.STL
- link ElbowLU_link: geometry collision mesh filename=package://arha_description/meshes/ElbowLU_link.STL; visual mesh filename=package://arha_description/meshes/ElbowLU_link.STL
- link ElbowRD_link: geometry collision mesh filename=package://arha_description/meshes/ElbowRD_link.STL; visual mesh filename=package://arha_description/meshes/ElbowRD_link.STL
- link ElbowRU_link: geometry collision mesh filename=package://arha_description/meshes/ElbowRU_link.STL; visual mesh filename=package://arha_description/meshes/ElbowRU_link.STL
- link ShoulderLD_link: geometry collision mesh filename=package://arha_description/meshes/ShoulderLD_link.STL; visual mesh filename=package://arha_description/meshes/ShoulderLD_link.STL
- link ShoulderLU_link: geometry collision mesh filename=package://arha_description/meshes/ShoulderLU_link.STL; visual mesh filename=package://arha_description/meshes/ShoulderLU_link.STL
- link ShoulderRD_link: geometry collision mesh filename=package://arha_description/meshes/ShoulderRD_link.STL; visual mesh filename=package://arha_description/meshes/ShoulderRD_link.STL
- link ShoulderRU_link: geometry collision mesh filename=package://arha_description/meshes/ShoulderRU_link.STL; visual mesh filename=package://arha_description/meshes/ShoulderRU_link.STL
- link WristLD_link: geometry collision mesh filename=package://arha_description/meshes/WristLD_link.STL; visual mesh filename=package://arha_description/meshes/WristLD_link.STL
- link WristLU_link: geometry collision mesh filename=package://arha_description/meshes/WristLU_link.STL; visual mesh filename=package://arha_description/meshes/WristLU_link.STL
- link WristRD_link: geometry collision mesh filename=package://arha_description/meshes/WristRD_link.STL; visual mesh filename=package://arha_description/meshes/WristRD_link.STL
- link WristRU_link: geometry collision mesh filename=package://arha_description/meshes/WristRU_link.STL; visual mesh filename=package://arha_description/meshes/WristRU_link.STL
Joints:
- joint ElbowLD_joint: limit lower=-1.5708 upper=0 effort=5000 velocity=4.1888 -> lower=-1.5708 upper=1.5708 effort=5000 velocity=4.1888
- joint ElbowRD_joint: limit lower=0 upper=1.5708 effort=5000 velocity=4.1888 -> lower=-1.5708 upper=1.5708 effort=5000 velocity=4.1888
- joint ShoulderLD_joint: limit lower=0 upper=1.5708 effort=5000 velocity=4.1888 -> lower=-1.5708 upper=1.5708 effort=5000 velocity=4.1888

File: arha_gazebo/urdf/arha_with_grippers.urdf.xacro (robot description, xacro)
@@ -2,21 +2,29 @@
 <robot xmlns:xacro="http://www.ros.org/wiki/xacro" name="arha_complete">
   <!-- Include base ARHA robot -->
-  <xacro:include filename="$(find arha_description)/urdf/ARHA.urdf"/>
-  <!-- Include left gripper -->
-  <xacro:include filename="$(find arha_gazebo)/urdf/grippers/left_gripper_mount.xacro"/>
-  <!-- Include right gripper -->
-  <xacro:include filename="$(find arha_gazebo)/urdf/grippers/right_gripper_mount.xacro"/>
-  <!-- Include wrist cameras -->
-  <xacro:include filename="$(find arha_gazebo)/urdf/sensors/camera_left_wrist.xacro"/>
-  <xacro:include filename="$(find arha_gazebo)/urdf/sensors/camera_right_wrist.xacro"/>
-  <!-- Include chest camera -->
+  <xacro:include filename="$(find arha_description)/urdf/ARHA_base.xacro"/>
+  <xacro:arha_base />
+  <!-- MoveIt2-aligned pincopen grippers + wrist cameras -->
+  <xacro:include filename="$(find arha_gazebo)/urdf/grippers/pincopen.xacro"/>
+  <xacro:include filename="$(find realsense2_description)/urdf/_d435.urdf.xacro"/>
+  <xacro:pincopen_gripper prefix="left" parent="WristLD_link">
+    <origin xyz="0 0 0.13" rpy="1.5708 -1.5708 3.14159" />
+  </xacro:pincopen_gripper>
+  <xacro:sensor_d435 parent="left_Camera_mount_V1" name="left_camera" use_nominal_extrinsics="false" add_plug="false" use_mesh="true">
+    <origin xyz="-0.01 -0.008 0.011" rpy="0 0 1.5708"/>
+  </xacro:sensor_d435>
+  <xacro:pincopen_gripper prefix="right" parent="WristRD_link">
+    <origin xyz="0 0 0.13" rpy="1.5708 -1.5708 0.0" />
+  </xacro:pincopen_gripper>
+  <xacro:sensor_d435 parent="right_Camera_mount_V1" name="right_camera" use_nominal_extrinsics="false" add_plug="false" use_mesh="true">
+    <origin xyz="-0.01 -0.008 0.011" rpy="0 0 1.5708"/>
+  </xacro:sensor_d435>
+  <!-- Keep head/chest camera -->
   <xacro:include filename="$(find arha_gazebo)/urdf/sensors/camera_chest.xacro"/>
-  <!-- Add world link for fixed base (temporary for testing) -->
+  <!-- Fixed base in Gazebo -->
   <link name="world"/>
-  <!-- Fix base_link to world -->
   <joint name="world_to_base" type="fixed">
     <parent link="world"/>
-    <child link="world_link"/>
-    <origin xyz="0 0 0" rpy="0 0 0"/>
+    <child link="base_link"/>
+    <origin xyz="0.15 0 0.00" rpy="0 0 0"/>
   </joint>
   <!-- Gazebo - Make base_link heavier and more stable -->
@@ -309,5 +317,5 @@
       <state_interface name="velocity"/>
     </joint>
-    <!-- Left Gripper Joints -->
+    <!-- Gripper actuation joints -->
     <joint name="left_cam_joint">
       <command_interface name="position">
@@ -315,8 +323,9 @@
         <param name="max">0.0</param>
       </command_interface>
-      <state_interface name="position"/>
-      <state_interface name="velocity"/>
-    </joint>
-    <!-- Right Gripper Joints -->
+      <state_interface name="position">
+        <param name="initial_value">-0.30</param>
+      </state_interface>
+      <state_interface name="velocity"/>
+    </joint>
     <joint name="right_cam_joint">
       <command_interface name="position">
@@ -324,4 +333,68 @@
         <param name="max">0.0</param>
       </command_interface>
+      <state_interface name="position">
+        <param name="initial_value">-0.30</param>
+      </state_interface>
+      <state_interface name="velocity"/>
+    </joint>
+    <!-- Left Gripper Mimic Joints -->
+    <joint name="left_Revolute_2_0">
+      <command_interface name="position"/>
+      <state_interface name="position"/>
+      <state_interface name="velocity"/>
+    </joint>
+    <joint name="left_Revolute_3_0">
+      <command_interface name="position"/>
+      <state_interface name="position"/>
+      <state_interface name="velocity"/>
+    </joint>
+    <joint name="left_Revolute_4_0">
+      <command_interface name="position"/>
+      <state_interface name="position"/>
+      <state_interface name="velocity"/>
+    </joint>
+    <joint name="left_Revolute_5_0">
+      <command_interface name="position"/>
+      <state_interface name="position"/>
+      <state_interface name="velocity"/>
+    </joint>
+    <joint name="left_Revolute_6_0">
+      <command_interface name="position"/>
+      <state_interface name="position"/>
+      <state_interface name="velocity"/>
+    </joint>
+    <joint name="left_Revolute_7_0">
+      <command_interface name="position"/>
+      <state_interface name="position"/>
+      <state_interface name="velocity"/>
+    </joint>
+    <!-- Right Gripper Mimic Joints -->
+    <joint name="right_Revolute_2_0">
+      <command_interface name="position"/>
+      <state_interface name="position"/>
+      <state_interface name="velocity"/>
+    </joint>
+    <joint name="right_Revolute_3_0">
+      <command_interface name="position"/>
+      <state_interface name="position"/>
+      <state_interface name="velocity"/>
+    </joint>
+    <joint name="right_Revolute_4_0">
+      <command_interface name="position"/>
+      <state_interface name="position"/>
+      <state_interface name="velocity"/>
+    </joint>
+    <joint name="right_Revolute_5_0">
+      <command_interface name="position"/>
+      <state_interface name="position"/>
+      <state_interface name="velocity"/>
+    </joint>
+    <joint name="right_Revolute_6_0">
+      <command_interface name="position"/>
+      <state_interface name="position"/>
+      <state_interface name="velocity"/>
+    </joint>
+    <joint name="right_Revolute_7_0">
+      <command_interface name="position"/>
       <state_interface name="position"/>
       <state_interface name="velocity"/>
@@ -333,6 +406,6 @@
       <ros>
         <namespace>/</namespace>
-        <argument>--ros-args</argument>
       </ros>
+      <robot_param_node>/robot_state_publisher/robot_state_publisher</robot_param_node>
       <parameters>$(find arha_gazebo)/config/gazebo_controllers.yaml</parameters>
     </plugin>

File: arha_gazebo/urdf/grippers/pincopen.xacro (robot description, xacro)
@@ -1,5 +1,5 @@
+<?xml version="1.0" ?>
 <robot xmlns:xacro="http://ros.org/wiki/xacro">
   <xacro:macro name="pincopen_gripper" params="prefix parent *origin">
-    <!-- Parent Attachment -->
     <joint name="${prefix}_gripper_mount_joint" type="fixed">
       <xacro:insert_block name="origin" />
@@ -8,4 +8,9 @@
     </joint>
     <link name="${prefix}_Bottom_Plate">
+        <inertial>
+            <mass value="0.500" />
+            <origin xyz="-0.0285975 -3.86746e-05 -0.00842464" rpy="0 0 0" />
+            <inertia ixx="2.5e-03" ixy="0" ixz="0" iyy="2.5e-03" iyz="0" izz="2.5e-03" />
+        </inertial>
         <visual>
             <geometry>
@@ -14,11 +19,11 @@
             <material name="light_grey"><color rgba="0.9 0.9 0.9 1" /></material>
         </visual>
-        <collision>
-            <geometry>
-                <mesh filename="package://pincopen/meshes/107.stl" scale="1 1 1" />
-            </geometry>
-        </collision>
     </link>
     <link name="${prefix}_Cam">
+        <inertial>
+            <mass value="0.100" />
+            <origin xyz="-9.28675e-06 -1.26037e-06 0.00337664" rpy="0 0 0" />
+            <inertia ixx="5.0e-04" ixy="0" ixz="0" iyy="5.0e-04" iyz="0" izz="5.0e-04" />
+        </inertial>
         <visual>
             <origin xyz="0.0180424 0 0.0024" rpy="0 -0 0" />
@@ -29,5 +34,4 @@
         </visual>
     </link>
-    <!-- Main Active Joint -->
     <joint name="${prefix}_cam_joint" type="revolute">
         <origin xyz="-0.0180424 0 -0.0035" rpy="0 0 -1.50657" />
@@ -35,8 +39,14 @@
         <parent link="${prefix}_Bottom_Plate" />
         <child link="${prefix}_Cam" />
+        <dynamics damping="10.0" friction="5.0"/>
         <limit effort="10" velocity="2.0" lower="-0.57" upper="0.0" />
     </joint>
-    <!-- Mimic Joints -->
+    <!-- ==================== FINGER 1 ==================== -->
     <link name="${prefix}_Internal_Rod_1">
+        <inertial>
+            <mass value="0.080" />
+            <origin xyz="0.0101857 0.0065898 0.008" rpy="0 0 0" />
+            <inertia ixx="3.0e-04" ixy="0" ixz="0" iyy="3.0e-04" iyz="0" izz="3.0e-04" />
+        </inertial>
         <visual>
             <origin xyz="0 0.0325 0.008" rpy="0 0 0" />
@@ -49,13 +59,40 @@
     <joint name="${prefix}_Revolute_2_0" type="revolute">
         <origin xyz="0 -0.0325 -0.0088" rpy="0 0 -0.0642" />
+        <parent link="${prefix}_Bottom_Plate" />
+        <child link="${prefix}_Internal_Rod_1" />
         <axis xyz="0 0 -1" />
-        <parent link="${prefix}_Bottom_Plate" />
-        <child link="${prefix}_Internal_Rod_1" />
-        <mimic joint="${prefix}_cam_joint" multiplier="-1.0" offset="0" />
-        <limit effort="10" velocity="2.0" lower="-1.57" upper="1.57" />
+        <limit effort="10" velocity="2.0" lower="-1.57" upper="1.57" />
+        <dynamics damping="1.0" friction="0.1"/>
+        <mimic joint="${prefix}_cam_joint" multiplier="-1.0" />
+    </joint>
+    <link name="${prefix}_External_Rod_1">
+        <inertial>
+            <mass value="0.060" />
+            <origin xyz="0.0173205 0.01 0.004" rpy="0 0 0" />
+            <inertia ixx="2.0e-04" ixy="0" ixz="0" iyy="2.0e-04" iyz="0" izz="2.0e-04" />
+        </inertial>
+        <visual>
+            <origin xyz="0 0.044 0.004" rpy="0 -0 0" />
+            <geometry><mesh filename="package://pincopen/meshes/119.stl" scale="1 1 1" /></geometry>
+            <material name="light_grey"/>
+        </visual>
+    </link>
+    <joint name="${prefix}_Revolute_4_0" type="revolute">
+        <origin xyz="0 -0.044 -0.0042" rpy="0 0 -0.0642296" />
+        <parent link="${prefix}_Bottom_Plate" />
+        <child link="${prefix}_External_Rod_1" />
+        <axis xyz="0 0 1" />
+        <limit effort="10" velocity="2.0" lower="-1.57" upper="1.57" />
+        <dynamics damping="1.0" friction="0.1"/>
+        <mimic joint="${prefix}_cam_joint" multiplier="1.0" />
     </joint>
     <link name="${prefix}_Distal_Rod">
-        <visual>
-            <origin xyz="-0.0346 0.0125 -0.0086" rpy="0 0 0" />
+        <inertial>
+            <mass value="0.060" />
+            <origin xyz="0.00258376 -0.00352926 -0.0086" rpy="0 0 0" />
+            <inertia ixx="2.0e-04" ixy="0" ixz="0" iyy="2.0e-04" iyz="0" izz="2.0e-04" />
+        </inertial>
+        <visual>
+            <origin xyz="-0.034641 0.0125 -0.0086" rpy="0 0 0" />
             <geometry>
                 <mesh filename="package://pincopen/meshes/63.stl" scale="1 1 1" />
@@ -65,12 +102,18 @@
     </link>
     <joint name="${prefix}_Revolute_5_0" type="revolute">
-        <origin xyz="0.0346 0.02 0.0165" rpy="0 0 0.0642" />
-        <axis xyz="0 0 1" />
+        <origin xyz="0.034641 0.02 0.0165" rpy="0 0 0.0642" />
         <parent link="${prefix}_Internal_Rod_1" />
         <child link="${prefix}_Distal_Rod" />
-        <mimic joint="${prefix}_cam_joint" multiplier="-1.0" offset="0" />
-        <limit effort="10" velocity="2.0" lower="-1.57" upper="1.57" />
+        <axis xyz="0 0 1" />
+        <limit effort="10" velocity="2.0" lower="-1.57" upper="1.57" />
+        <dynamics damping="1.0" friction="0.1"/>
+        <mimic joint="${prefix}_cam_joint" multiplier="-1.0" />
     </joint>
     <link name="${prefix}_Removable_Tip_1">
+        <inertial>
+            <mass value="0.040" />
+            <origin xyz="0.00745849 0.0018564 -0.0049" rpy="0 0 0" />
+            <inertia ixx="1.5e-04" ixy="0" ixz="0" iyy="1.5e-04" iyz="0" izz="1.5e-04" />
+        </inertial>
         <visual>
             <origin xyz="-0.0428 0.0147 -0.0049" rpy="0 0 0" />
@@ -78,10 +121,12 @@
                 <mesh filename="package://pincopen/meshes/123.stl" scale="1 1 1" />
             </geometry>
-            <material name="light_grey"/>
+            <material name="finger_tip_dark">
+                <color rgba="0.15 0.15 0.15 1" />
+            </material>
         </visual>
         <collision>
             <origin xyz="-0.0428 0.0147 -0.0049" rpy="0 0 0" />
             <geometry>
-                <mesh filename="package://pincopen/meshes/123.stl" scale="1 1 1" />
+                <box size="0.02 0.01 0.01" />
             </geometry>
         </collision>
@@ -92,5 +137,11 @@
         <child link="${prefix}_Removable_Tip_1" />
     </joint>
+    <!-- ==================== FINGER 2 ==================== -->
     <link name="${prefix}_Internal_Rod">
+        <inertial>
+            <mass value="0.080" />
+            <origin xyz="0.0101857 0.0065898 -0.008" rpy="0 0 0" />
+            <inertia ixx="3.0e-04" ixy="0" ixz="0" iyy="3.0e-04" iyz="0" izz="3.0e-04" />
+        </inertial>
         <visual>
             <origin xyz="0 0.0325 -0.008" rpy="0 0 0" />
@@ -103,13 +154,40 @@
     <joint name="${prefix}_Revolute_3_0" type="revolute">
         <origin xyz="0 0.0325 -0.0088" rpy="3.14159 0 0.0642" />
+        <parent link="${prefix}_Bottom_Plate" />
+        <child link="${prefix}_Internal_Rod" />
         <axis xyz="0 0 1" />
-        <parent link="${prefix}_Bottom_Plate" />
-        <child link="${prefix}_Internal_Rod" />
-        <mimic joint="${prefix}_cam_joint" multiplier="1.0" offset="0" />
-        <limit effort="10" velocity="2.0" lower="-1.57" upper="1.57" />
+        <limit effort="10" velocity="2.0" lower="-1.57" upper="1.57" />
+        <dynamics damping="1.0" friction="0.1"/>
+        <mimic joint="${prefix}_cam_joint" multiplier="1.0" />
+    </joint>
+    <link name="${prefix}_External_Rod">
+        <inertial>
+            <mass value="0.060" />
+            <origin xyz="0.0173205 0.01 0.004" rpy="0 0 0" />
+            <inertia ixx="2.0e-04" ixy="0" ixz="0" iyy="2.0e-04" iyz="0" izz="2.0e-04" />
+        </inertial>
+        <visual>
+            <origin xyz="0 0.044 0.004" rpy="0 -0 0" />
+            <geometry><mesh filename="package://pincopen/meshes/79.stl" scale="1 1 1" /></geometry>
+            <material name="light_grey"/>
+        </visual>
+    </link>
+    <joint name="${prefix}_Revolute_6_0" type="revolute">
+        <origin xyz="0 0.044 -0.0042" rpy="0 0 -0.982968" />
+        <parent link="${prefix}_Bottom_Plate" />
+        <child link="${prefix}_External_Rod" />
+        <axis xyz="0 0 1" />
+        <limit effort="10" velocity="2.0" lower="-1.57" upper="1.57" />
+        <dynamics damping="1.0" friction="0.1"/>
+        <mimic joint="${prefix}_cam_joint" multiplier="-1.0" />
     </joint>
     <link name="${prefix}_Distal_Rod_1">
-        <visual>
-            <origin xyz="-0.0346 0.0125 0.0086" rpy="0 0 0" />
+        <inertial>
+            <mass value="0.060" />
+            <origin xyz="0.00258376 -0.00352926 0.0086" rpy="0 0 0" />
+            <inertia ixx="2.0e-04" ixy="0" ixz="0" iyy="2.0e-04" iyz="0" izz="2.0e-04" />
+        </inertial>
+        <visual>
+            <origin xyz="-0.034641 0.0125 0.0086" rpy="0 0 0" />
             <geometry>
                 <mesh filename="package://pincopen/meshes/71.stl" scale="1 1 1" />
@@ -119,12 +197,18 @@
     </link>
     <joint name="${prefix}_Revolute_7_0" type="revolute">
-        <origin xyz="0.0346 0.02 -0.0165" rpy="0 0 0.0642" />
-        <axis xyz="0 0 -1" />
+        <origin xyz="0.034641 0.02 -0.0165" rpy="0 0 0.0642" />
         <parent link="${prefix}_Internal_Rod" />
         <child link="${prefix}_Distal_Rod_1" />
-        <mimic joint="${prefix}_cam_joint" multiplier="1.0" offset="0" />
-        <limit effort="10" velocity="2.0" lower="-1.57" upper="1.57" />
+        <axis xyz="0 0 -1" />
+        <limit effort="10" velocity="2.0" lower="-1.57" upper="1.57" />
+        <dynamics damping="1.0" friction="0.1"/>
+        <mimic joint="${prefix}_cam_joint" multiplier="1.0" />
     </joint>
     <link name="${prefix}_Removable_Tip">
+        <inertial>
+            <mass value="0.040" />
+            <origin xyz="0.00745849 0.0018564 0.0049" rpy="0 0 0" />
+            <inertia ixx="1.5e-04" ixy="0" ixz="0" iyy="1.5e-04" iyz="0" izz="1.5e-04" />
+        </inertial>
         <visual>
             <origin xyz="-0.0428 0.0147 0.0049" rpy="0 0 0" />
@@ -132,10 +216,12 @@
                 <mesh filename="package://pincopen/meshes/83.stl" scale="1 1 1" />
             </geometry>
-            <material name="light_grey"/>
+            <material name="finger_tip_dark">
+                <color rgba="0.15 0.15 0.15 1" />
+            </material>
         </visual>
         <collision>
             <origin xyz="-0.0428 0.0147 0.0049" rpy="0 0 0" />
             <geometry>
-                <mesh filename="package://pincopen/meshes/83.stl" scale="1 1 1" />
+                <box size="0.02 0.01 0.01" />
             </geometry>
         </collision>
@@ -146,4 +232,5 @@
         <child link="${prefix}_Removable_Tip" />
     </joint>
+    <!-- ==================== STATIC ATTACHMENTS ==================== -->
     <link name="${prefix}_Top_Plate">
         <visual>
@@ -230,39 +317,16 @@
         <child link="${prefix}_Distal_Shell_1" />
     </joint>
-    <link name="${prefix}_External_Rod">
-        <visual>
-            <origin xyz="0 0.044 0.004" rpy="0 -0 0" />
-            <geometry><mesh filename="package://pincopen/meshes/79.stl" scale="1 1 1" /></geometry>
-            <material name="light_grey"/>
-        </visual>
-    </link>
-    <joint name="${prefix}_Revolute_6_0" type="revolute">
-        <origin xyz="0 0.044 -0.0042" rpy="0 0 -0.982968" />
-        <axis xyz="0 0 1" />
-        <parent link="${prefix}_Bottom_Plate" />
-        <child link="${prefix}_External_Rod" />
-        <mimic joint="${prefix}_cam_joint" multiplier="-1.0" offset="0" />
-        <limit effort="10" velocity="2.0" lower="-1.57" upper="1.57" />
-    </joint>
-    <link name="${prefix}_External_Rod_1">
-        <visual>
-            <origin xyz="0 0.044 0.004" rpy="0 -0 0" />
-            <geometry><mesh filename="package://pincopen/meshes/119.stl" scale="1 1 1" /></geometry>
-            <material name="light_grey"/>
-        </visual>
-    </link>
-    <joint name="${prefix}_Revolute_4_0" type="revolute">
-        <origin xyz="0 -0.044 -0.0042" rpy="0 0 -0.0642296" />
-        <axis xyz="0 0 1" />
-        <parent link="${prefix}_Bottom_Plate" />
-        <child link="${prefix}_External_Rod_1" />
-        <mimic joint="${prefix}_cam_joint" multiplier="1.0" offset="0" />
-        <limit effort="10" velocity="2.0" lower="-1.57" upper="1.57" />
-    </joint>
     <link name="${prefix}_Tip_Support">
+        <inertial>
+            <mass value="0.030" />
+            <origin xyz="0.00385164 0.0032358 0.00350015" rpy="0 0 0" />
+            <inertia ixx="1.0e-04" ixy="0" ixz="0" iyy="1.0e-04" iyz="0" izz="1.0e-04" />
+        </inertial>
         <visual>
             <origin xyz="-0.051641 0.00775 0.0035" rpy="0 -0 0" />
             <geometry><mesh filename="package://pincopen/meshes/95.stl" scale="1 1 1" /></geometry>
-            <material name="light_grey"/>
+            <material name="finger_support_dark">
+                <color rgba="0.25 0.25 0.25 1" />
+            </material>
         </visual>
     </link>
@@ -273,8 +337,15 @@
     </joint>
     <link name="${prefix}_Tip_Support_1">
+        <inertial>
+            <mass value="0.030" />
+            <origin xyz="0.00385164 0.0032358 -0.00349985" rpy="0 0 0" />
+            <inertia ixx="1.0e-04" ixy="0" ixz="0" iyy="1.0e-04" iyz="0" izz="1.0e-04" />
+        </inertial>
         <visual>
             <origin xyz="-0.051641 0.00775 -0.0035" rpy="0 -0 0" />
             <geometry><mesh filename="package://pincopen/meshes/99.stl" scale="1 1 1" /></geometry>
-            <material name="light_grey"/>
+            <material name="finger_support_dark">
+                <color rgba="0.25 0.25 0.25 1" />
+            </material>
         </visual>
     </link>
@@ -284,4 +355,6 @@
         <child link="${prefix}_Tip_Support_1" />
     </joint>
+    <!-- Note - Mimic joint behavior is handled by gazebo_ros2_control which reads
+         the <mimic> tags from URDF. The mimic plugins are no longer needed. -->
   </xacro:macro>
 </robot>
