Commit message: refactor: changes related to gazebo and moveit2 for virtual simulation of new grippers and controllers.

File: arha_gazebo/urdf/sensors/camera_left_wrist.xacro (robot description, xacro)
@@ -4,5 +4,5 @@
   <xacro:include filename="$(find realsense2_description)/urdf/_d435.urdf.xacro"/>
   <!-- Instantiate RealSense D435 on left gripper link -->
-  <xacro:sensor_d435 parent="left_robotiq_hande_link" name="camera_left_wrist" use_nominal_extrinsics="true">
+  <xacro:sensor_d435 parent="WristLD_link" name="camera_left_wrist" use_nominal_extrinsics="true">
     <!-- Position - slightly to the side and forward of gripper -->
     <origin xyz="0.0 0.075 0.0005" rpy="0 -1.5708 1.5708"/>

File: arha_gazebo/urdf/sensors/camera_right_wrist.xacro (robot description, xacro)
@@ -4,5 +4,5 @@
   <xacro:include filename="$(find realsense2_description)/urdf/_d435.urdf.xacro"/>
   <!-- Instantiate RealSense D435 directly on gripper link -->
-  <xacro:sensor_d435 parent="right_robotiq_hande_link" name="camera_right_wrist" use_nominal_extrinsics="true">
+  <xacro:sensor_d435 parent="WristRD_link" name="camera_right_wrist" use_nominal_extrinsics="true">
     <!-- Position - slightly to the side and forward of gripper -->
     <origin xyz="0.0 -0.075 0.0005" rpy="0 -1.5708 -1.5708"/>

File: arha_moveit2/config/arha_description.ros2_control.xacro (robot description, xacro)
@@ -167,4 +167,40 @@
                 <param name="direction">1</param>
             </joint>
+            <joint name="left_Revolute_2_0">
+                <param name="mimic">left_cam_joint</param>
+                <param name="multiplier">1.0</param>
+                <command_interface name="position"/>
+                <state_interface name="position"/>
+            </joint>
+            <joint name="left_Revolute_4_0">
+                <param name="mimic">left_cam_joint</param>
+                <param name="multiplier">-1.0</param>
+                <command_interface name="position"/>
+                <state_interface name="position"/>
+            </joint>
+            <joint name="left_Revolute_5_0">
+                <param name="mimic">left_cam_joint</param>
+                <param name="multiplier">-1.0</param>
+                <command_interface name="position"/>
+                <state_interface name="position"/>
+            </joint>
+            <joint name="left_Revolute_3_0">
+                <param name="mimic">left_cam_joint</param>
+                <param name="multiplier">1.0</param>
+                <command_interface name="position"/>
+                <state_interface name="position"/>
+            </joint>
+            <joint name="left_Revolute_6_0">
+                <param name="mimic">left_cam_joint</param>
+                <param name="multiplier">-1.0</param>
+                <command_interface name="position"/>
+                <state_interface name="position"/>
+            </joint>
+            <joint name="left_Revolute_7_0">
+                <param name="mimic">left_cam_joint</param>
+                <param name="multiplier">-1.0</param>
+                <command_interface name="position"/>
+                <state_interface name="position"/>
+            </joint>
             <joint name="right_cam_joint">
                 <command_interface name="position"/>
@@ -178,4 +214,40 @@
                 <param name="direction">1</param>
             </joint>
+            <joint name="right_Revolute_2_0">
+                <param name="mimic">right_cam_joint</param>
+                <param name="multiplier">1.0</param>
+                <command_interface name="position"/>
+                <state_interface name="position"/>
+            </joint>
+            <joint name="right_Revolute_4_0">
+                <param name="mimic">right_cam_joint</param>
+                <param name="multiplier">-1.0</param>
+                <command_interface name="position"/>
+                <state_interface name="position"/>
+            </joint>
+            <joint name="right_Revolute_5_0">
+                <param name="mimic">right_cam_joint</param>
+                <param name="multiplier">-1.0</param>
+                <command_interface name="position"/>
+                <state_interface name="position"/>
+            </joint>
+            <joint name="right_Revolute_3_0">
+                <param name="mimic">right_cam_joint</param>
+                <param name="multiplier">1.0</param>
+                <command_interface name="position"/>
+                <state_interface name="position"/>
+            </joint>
+            <joint name="right_Revolute_6_0">
+                <param name="mimic">right_cam_joint</param>
+                <param name="multiplier">-1.0</param>
+                <command_interface name="position"/>
+                <state_interface name="position"/>
+            </joint>
+            <joint name="right_Revolute_7_0">
+                <param name="mimic">right_cam_joint</param>
+                <param name="multiplier">-1.0</param>
+                <command_interface name="position"/>
+                <state_interface name="position"/>
+            </joint>
         </ros2_control>
     </xacro:macro>

File: arha_moveit2/config/arha_description.ros2_control_right_arm.xacro (robot description, xacro)
@@ -94,4 +94,40 @@
                 <param name="direction">1</param>
             </joint>
+            <joint name="right_Revolute_2_0">
+                <param name="mimic">right_cam_joint</param>
+                <param name="multiplier">1.0</param>
+                <command_interface name="position"/>
+                <state_interface name="position"/>
+            </joint>
+            <joint name="right_Revolute_4_0">
+                <param name="mimic">right_cam_joint</param>
+                <param name="multiplier">-1.0</param>
+                <command_interface name="position"/>
+                <state_interface name="position"/>
+            </joint>
+            <joint name="right_Revolute_5_0">
+                <param name="mimic">right_cam_joint</param>
+                <param name="multiplier">-1.0</param>
+                <command_interface name="position"/>
+                <state_interface name="position"/>
+            </joint>
+            <joint name="right_Revolute_3_0">
+                <param name="mimic">right_cam_joint</param>
+                <param name="multiplier">1.0</param>
+                <command_interface name="position"/>
+                <state_interface name="position"/>
+            </joint>
+            <joint name="right_Revolute_6_0">
+                <param name="mimic">right_cam_joint</param>
+                <param name="multiplier">-1.0</param>
+                <command_interface name="position"/>
+                <state_interface name="position"/>
+            </joint>
+            <joint name="right_Revolute_7_0">
+                <param name="mimic">right_cam_joint</param>
+                <param name="multiplier">-1.0</param>
+                <command_interface name="position"/>
+                <state_interface name="position"/>
+            </joint>
         </ros2_control>
     </xacro:macro>
