Commit message: adding new updated code

File: arha_moveit2/config/arha_description.ros2_control.xacro (robot description, xacro)
@@ -1,11 +1,19 @@
 <?xml version="1.0"?>
 <robot xmlns:xacro="http://www.ros.org/wiki/xacro">
-    <xacro:macro name="arha_description_ros2_control" params="name initial_positions_file">
+    <xacro:macro name="arha_description_ros2_control" params="name initial_positions_file use_fake_hardware:=true zero_on_startup:=false">
         <xacro:property name="initial_positions" value="${load_yaml(initial_positions_file)['initial_positions']}"/>
         <ros2_control name="${name}" type="system">
             <hardware>
-                <!-- By default, set up controllers for simulation. This won't work on real hardware -->
-                <plugin>mock_components/GenericSystem</plugin>
+                <xacro:if value="${use_fake_hardware}">
+                    <plugin>mock_components/GenericSystem</plugin>
+                </xacro:if>
+                <xacro:unless value="${use_fake_hardware}">
+                    <plugin>arha_hardware_interface/ArhaHardwareInterface</plugin>
+                    <param name="ip_address">192.168.197.123</param>
+                    <param name="port">5000</param>
+                    <param name="zero_on_startup">${zero_on_startup}</param>
+                </xacro:unless>
             </hardware>
+            <!-- LEFT ARM JOINTS -->
             <joint name="ShoulderLU_joint">
                 <command_interface name="position"/>
@@ -14,4 +22,8 @@
                 </state_interface>
                 <state_interface name="velocity"/>
+                <state_interface name="effort"/>
+                <param name="limb_name">left_arm</param>
+                <param name="motor_id">1</param>
+                <param name="direction">-1</param>
             </joint>
             <joint name="ShoulderLD_joint">
@@ -21,4 +33,8 @@
                 </state_interface>
                 <state_interface name="velocity"/>
+                <state_interface name="effort"/>
+                <param name="limb_name">left_arm</param>
+                <param name="motor_id">2</param>
+                <param name="direction">-1</param>
             </joint>
             <joint name="ElbowLU_joint">
@@ -28,4 +44,8 @@
                 </state_interface>
                 <state_interface name="velocity"/>
+                <state_interface name="effort"/>
+                <param name="limb_name">left_arm</param>
+                <param name="motor_id">3</param>
+                <param name="direction">-1</param>
             </joint>
             <joint name="ElbowLD_joint">
@@ -35,4 +55,8 @@
                 </state_interface>
                 <state_interface name="velocity"/>
+                <state_interface name="effort"/>
+                <param name="limb_name">left_arm</param>
+                <param name="motor_id">4</param>
+                <param name="direction">-1</param>
             </joint>
             <joint name="WristLU_joint">
@@ -42,4 +66,8 @@
                 </state_interface>
                 <state_interface name="velocity"/>
+                <state_interface name="effort"/>
+                <param name="limb_name">left_arm</param>
+                <param name="motor_id">5</param>
+                <param name="direction">-1</param>
             </joint>
             <joint name="WristLD_joint">
@@ -49,5 +77,10 @@
                 </state_interface>
                 <state_interface name="velocity"/>
+                <state_interface name="effort"/>
+                <param name="limb_name">left_arm</param>
+                <param name="motor_id">6</param>
+                <param name="direction">-1</param>
             </joint>
+            <!-- RIGHT ARM JOINTS -->
             <joint name="ShoulderRU_joint">
                 <command_interface name="position"/>
@@ -56,4 +89,8 @@
                 </state_interface>
                 <state_interface name="velocity"/>
+                <state_interface name="effort"/>
+                <param name="limb_name">right_arm</param>
+                <param name="motor_id">1</param>
+                <param name="direction">-1</param>
             </joint>
             <joint name="ShoulderRD_joint">
@@ -63,4 +100,8 @@
                 </state_interface>
                 <state_interface name="velocity"/>
+                <state_interface name="effort"/>
+                <param name="limb_name">right_arm</param>
+                <param name="motor_id">2</param>
+                <param name="direction">-1</param>
             </joint>
             <joint name="ElbowRU_joint">
@@ -70,4 +111,8 @@
                 </state_interface>
                 <state_interface name="velocity"/>
+                <state_interface name="effort"/>
+                <param name="limb_name">right_arm</param>
+                <param name="motor_id">3</param>
+                <param name="direction">-1</param>
             </joint>
             <joint name="ElbowRD_joint">
@@ -77,4 +122,8 @@
                 </state_interface>
                 <state_interface name="velocity"/>
+                <state_interface name="effort"/>
+                <param name="limb_name">right_arm</param>
+                <param name="motor_id">4</param>
+                <param name="direction">-1</param>
             </joint>
             <joint name="WristRU_joint">
@@ -84,4 +133,8 @@
                 </state_interface>
                 <state_interface name="velocity"/>
+                <state_interface name="effort"/>
+                <param name="limb_name">right_arm</param>
+                <param name="motor_id">5</param>
+                <param name="direction">-1</param>
             </joint>
             <joint name="WristRD_joint">
@@ -91,4 +144,8 @@
                 </state_interface>
                 <state_interface name="velocity"/>
+                <state_interface name="effort"/>
+                <param name="limb_name">right_arm</param>
+                <param name="motor_id">6</param>
+                <param name="direction">-1</param>
             </joint>
         </ros2_control>

File: arha_moveit2/config/arha_description.urdf.xacro (robot description, xacro)
@@ -2,8 +2,10 @@
 <robot xmlns:xacro="http://www.ros.org/wiki/xacro" name="arha_description">
     <xacro:arg name="initial_positions_file" default="initial_positions.yaml" />
+    <xacro:arg name="use_fake_hardware" default="true" />
+    <xacro:arg name="zero_on_startup" default="false" />
     <!-- Import arha_description urdf file -->
     <xacro:include filename="$(find arha_description)/urdf/ARHA.urdf" />
     <!-- Import control_xacro -->
     <xacro:include filename="arha_description.ros2_control.xacro" />
-    <xacro:arha_description_ros2_control name="FakeSystem" initial_positions_file="$(arg initial_positions_file)"/>
+    <xacro:arha_description_ros2_control name="ARHA" initial_positions_file="$(arg initial_positions_file)" use_fake_hardware="$(arg use_fake_hardware)" zero_on_startup="$(arg zero_on_startup)"/>
 </robot>

Commit message: adding fixes to some files

File: arha_moveit2/config/arha_description.ros2_control.xacro (robot description, xacro)
@@ -164,42 +164,6 @@
                 <state_interface name="effort"/>
                 <param name="limb_name">left_gripper</param>
-                <param name="motor_id">2</param>
+                <param name="motor_id">1</param>
                 <param name="direction">1</param>
-            </joint>
-            <joint name="left_Revolute_2_0">
-                <param name="mimic">left_cam_joint</param>
-                <param name="multiplier">1.0</param>
-                <command_interface name="position"/>
-                <state_interface name="position"/>
-            </joint>
-            <joint name="left_Revolute_4_0">
-                <param name="mimic">left_cam_joint</param>
-                <param name="multiplier">-1.0</param>
-                <command_interface name="position"/>
-                <state_interface name="position"/>
-            </joint>
-            <joint name="left_Revolute_5_0">
-                <param name="mimic">left_cam_joint</param>
-                <param name="multiplier">-1.0</param>
-                <command_interface name="position"/>
-                <state_interface name="position"/>
-            </joint>
-            <joint name="left_Revolute_3_0">
-                <param name="mimic">left_cam_joint</param>
-                <param name="multiplier">1.0</param>
-                <command_interface name="position"/>
-                <state_interface name="position"/>
-            </joint>
-            <joint name="left_Revolute_6_0">
-                <param name="mimic">left_cam_joint</param>
-                <param name="multiplier">-1.0</param>
-                <command_interface name="position"/>
-                <state_interface name="position"/>
-            </joint>
-            <joint name="left_Revolute_7_0">
-                <param name="mimic">left_cam_joint</param>
-                <param name="multiplier">-1.0</param>
-                <command_interface name="position"/>
-                <state_interface name="position"/>
             </joint>
             <joint name="right_cam_joint">
@@ -211,42 +175,6 @@
                 <state_interface name="effort"/>
                 <param name="limb_name">right_gripper</param>
-                <param name="motor_id">1</param>
+                <param name="motor_id">2</param>
                 <param name="direction">1</param>
-            </joint>
-            <joint name="right_Revolute_2_0">
-                <param name="mimic">right_cam_joint</param>
-                <param name="multiplier">1.0</param>
-                <command_interface name="position"/>
-                <state_interface name="position"/>
-            </joint>
-            <joint name="right_Revolute_4_0">
-                <param name="mimic">right_cam_joint</param>
-                <param name="multiplier">-1.0</param>
-                <command_interface name="position"/>
-                <state_interface name="position"/>
-            </joint>
-            <joint name="right_Revolute_5_0">
-                <param name="mimic">right_cam_joint</param>
-                <param name="multiplier">-1.0</param>
-                <command_interface name="position"/>
-                <state_interface name="position"/>
-            </joint>
-            <joint name="right_Revolute_3_0">
-                <param name="mimic">right_cam_joint</param>
-                <param name="multiplier">1.0</param>
-                <command_interface name="position"/>
-                <state_interface name="position"/>
-            </joint>
-            <joint name="right_Revolute_6_0">
-                <param name="mimic">right_cam_joint</param>
-                <param name="multiplier">-1.0</param>
-                <command_interface name="position"/>
-                <state_interface name="position"/>
-            </joint>
-            <joint name="right_Revolute_7_0">
-                <param name="mimic">right_cam_joint</param>
-                <param name="multiplier">-1.0</param>
-                <command_interface name="position"/>
-                <state_interface name="position"/>
             </joint>
         </ros2_control>

File: arha_moveit2/config/arha_description.ros2_control_right_arm.xacro (robot description, xacro)
@@ -13,4 +13,9 @@
                     <param name="port">5000</param>
                     <param name="zero_on_startup">false</param>
+                    <!-- Gravity Compensation Required Params -->
+                    <param name="gravity_compensation">true</param>
+                    <param name="urdf_path">$(find arha_description)/urdf/ARHA.urdf</param>
+                    <param name="right_arm_base_link">chest_link</param>
+                    <param name="right_arm_tip_link">WristRD_link</param>
                 </xacro:unless>
             </hardware>
@@ -80,5 +85,5 @@
                 <param name="limb_name">right_arm</param>
                 <param name="motor_id">6</param>
-                <param name="direction">1</param>
+                <param name="direction">-1</param>
             </joint>
             <!-- Gripper -->
@@ -91,10 +96,10 @@
                 <state_interface name="effort"/>
                 <param name="limb_name">right_gripper</param>
-                <param name="motor_id">1</param>
+                <param name="motor_id">2</param>
                 <param name="direction">1</param>
             </joint>
             <joint name="right_Revolute_2_0">
                 <param name="mimic">right_cam_joint</param>
-                <param name="multiplier">1.0</param>
+                <param name="multiplier">-1.0</param>
                 <command_interface name="position"/>
                 <state_interface name="position"/>
@@ -102,5 +107,5 @@
             <joint name="right_Revolute_4_0">
                 <param name="mimic">right_cam_joint</param>
-                <param name="multiplier">-1.0</param>
+                <param name="multiplier">1.0</param>
                 <command_interface name="position"/>
                 <state_interface name="position"/>
@@ -126,5 +131,5 @@
             <joint name="right_Revolute_7_0">
                 <param name="mimic">right_cam_joint</param>
-                <param name="multiplier">-1.0</param>
+                <param name="multiplier">1.0</param>
                 <command_interface name="position"/>
                 <state_interface name="position"/>

File: arha_moveit2/config/arha_description.urdf.xacro (robot description, xacro)
@@ -7,5 +7,5 @@
     <xacro:include filename="$(find arha_description)/urdf/ARHA.urdf" />
     <!-- Gripper and Camera Assembly -->
-    <xacro:include filename="$(find arha_gazebo)/urdf/grippers/pincopen.xacro"/>
+    <xacro:include filename="$(find arha_moveit2)/config/grippers/pincopen_stub.xacro"/>
     <xacro:include filename="$(find realsense2_description)/urdf/_d435.urdf.xacro" />
     <xacro:pincopen_gripper prefix="left" parent="WristLD_link">

File: arha_moveit2/config/arha_description_right_arm.urdf.xacro (robot description, xacro)
@@ -6,5 +6,10 @@
     <xacro:include filename="$(find arha_description)/urdf/ARHA.urdf" />
     <!-- Gripper and Camera Assembly -->
-    <xacro:include filename="$(find arha_gazebo)/urdf/grippers/pincopen.xacro"/>
+    <xacro:if value="$(arg use_fake_hardware)">
+      <xacro:include filename="$(find arha_gazebo)/urdf/grippers/pincopen.xacro"/>
+    </xacro:if>
+    <xacro:unless value="$(arg use_fake_hardware)">
+      <xacro:include filename="$(find arha_moveit2)/config/grippers/pincopen_stub.xacro"/>
+    </xacro:unless>
     <xacro:include filename="$(find realsense2_description)/urdf/_d435.urdf.xacro" />
     <xacro:pincopen_gripper prefix="right" parent="WristRD_link">
