Commit message: Integrated head assembly with D435 camera and resolved SRDF collision matrix

File: arha_gazebo/urdf/arha_with_grippers.urdf.xacro (robot description, xacro)
@@ -7,4 +7,14 @@
   <xacro:include filename="$(find arha_gazebo)/urdf/grippers/pincopen.xacro"/>
   <xacro:include filename="$(find realsense2_description)/urdf/_d435.urdf.xacro"/>
+  <!-- Add the Head assembly -->
+  <xacro:include filename="$(find head)/urdf/head.xacro"/>
+  <!-- Raised head slightly higher (z=0.25) to ensure it clears the chest bounding box visibly -->
+  <xacro:arha_head parent="chest_link">
+    <origin xyz="-0.1 0 0.08" rpy="0 0 0" />
+  </xacro:arha_head>
+  <!-- Mount D435 Camera to the Head -->
+  <xacro:sensor_d435 parent="head_part_1_4" name="head_camera" use_nominal_extrinsics="false" add_plug="false" use_mesh="true">
+    <origin xyz="-0.18 -0.12 -0.037" rpy="1.5708 0 -1.5708"/>
+  </xacro:sensor_d435>
   <xacro:pincopen_gripper prefix="left" parent="WristLD_link">
     <origin xyz="0 0 0.13" rpy="1.5708 -1.5708 3.14159" />
@@ -19,6 +29,4 @@
     <origin xyz="-0.01 -0.008 0.011" rpy="0 0 1.5708"/>
   </xacro:sensor_d435>
-  <!-- Keep head/chest camera -->
-  <xacro:include filename="$(find arha_gazebo)/urdf/sensors/camera_chest.xacro"/>
   <!-- Fixed base in Gazebo -->
   <link name="world"/>

File: arha_moveit2/config/arha_description.urdf.xacro (robot description, xacro)
@@ -9,4 +9,13 @@
     <xacro:include filename="$(find arha_moveit2)/config/grippers/pincopen_stub.xacro"/>
     <xacro:include filename="$(find realsense2_description)/urdf/_d435.urdf.xacro" />
+    <!-- Add the Head assembly -->
+    <xacro:include filename="$(find head)/urdf/head.xacro"/>
+    <xacro:arha_head parent="chest_link">
+      <origin xyz="-0.1 0 0.08" rpy="0 0 0" />
+    </xacro:arha_head>
+    <!-- Mount D435 Camera to the Head -->
+    <xacro:sensor_d435 parent="head_part_1_4" name="head_camera" use_nominal_extrinsics="false" add_plug="false" use_mesh="true">
+      <origin xyz="-0.18 -0.12 -0.037" rpy="1.5708 0 -1.5708"/>
+    </xacro:sensor_d435>
     <xacro:pincopen_gripper prefix="left" parent="WristLD_link">
       <origin xyz="0 0 0.13" rpy="1.5708 -1.5708 3.14159" />

File: arha_moveit2/config/arha_description_right_arm.urdf.xacro (robot description, xacro)
@@ -13,4 +13,13 @@
     </xacro:unless>
     <xacro:include filename="$(find realsense2_description)/urdf/_d435.urdf.xacro" />
+    <!-- Add the Head assembly -->
+    <xacro:include filename="$(find head)/urdf/head.xacro"/>
+    <xacro:arha_head parent="chest_link">
+      <origin xyz="-0.1 0 0.08" rpy="0 0 0" />
+    </xacro:arha_head>
+    <!-- Mount D435 Camera to the Head -->
+    <xacro:sensor_d435 parent="head_part_1_4" name="head_camera" use_nominal_extrinsics="false" add_plug="false" use_mesh="true">
+      <origin xyz="-0.18 -0.12 -0.037" rpy="1.5708 0 -1.5708"/>
+    </xacro:sensor_d435>
     <xacro:pincopen_gripper prefix="right" parent="WristRD_link">
       <origin xyz="0 0 0.13" rpy="1.5708 -1.5708 0.0" />
